Commit message: Fix gripper motion planning: mimic joint URDF fixes, full joint_limits.yaml integration, and MoveIt config update

File: kortex_description/grippers/gen3_lite_2f/urdf/gen3_lite_2f.ros2_control.xacro (robot description, xacro)
@@ -66,31 +66,29 @@
             <!-- When simulating we need to include the rest of the gripper joints -->
             <xacro:if value="${use_fake_hardware or sim_isaac or sim_gazebo}">
-                <joint name="${prefix}right_finger_tip_joint">
-                    <param name="mimic">${prefix}right_finger_bottom_joint</param>
-                    <param name="multiplier">-1</param>
-                    <xacro:unless value="${sim_gazebo}">
-                        <command_interface name="position"/>
-                        <state_interface name="position"/>
-                        <state_interface name="velocity"/>
-                    </xacro:unless>
-                </joint>
-                <joint name="${prefix}left_finger_bottom_joint">
-                    <param name="mimic">${prefix}right_finger_bottom_joint</param>
-                    <param name="multiplier">-1</param>
-                    <xacro:unless value="${sim_gazebo}">
-                        <command_interface name="position"/>
-                        <state_interface name="position"/>
-                        <state_interface name="velocity"/>
-                    </xacro:unless>
-                </joint>
-                <joint name="${prefix}left_finger_tip_joint">
-                    <param name="mimic">${prefix}right_finger_bottom_joint</param>
-                    <param name="multiplier">-1</param>
-                    <xacro:unless value="${sim_gazebo}">
-                        <command_interface name="position"/>
-                        <state_interface name="position"/>
-                        <state_interface name="velocity"/>
-                    </xacro:unless>
-                </joint>
+                <!-- Always define mimic joints -->
+                    <joint name="${prefix}right_finger_tip_joint">
+                        <param name="mimic">${prefix}right_finger_bottom_joint</param>
+                        <param name="multiplier">-1</param>
+                        <xacro:if value="${use_fake_hardware or sim_isaac or sim_gazebo}">
+                            <state_interface name="position"/>
+                            <state_interface name="velocity"/>
+                        </xacro:if>
+                    </joint>
+                    <joint name="${prefix}left_finger_bottom_joint">
+                        <param name="mimic">${prefix}right_finger_bottom_joint</param>
+                        <param name="multiplier">-1</param>
+                        <xacro:if value="${use_fake_hardware or sim_isaac or sim_gazebo}">
+                            <state_interface name="position"/>
+                            <state_interface name="velocity"/>
+                        </xacro:if>
+                    </joint>
+                    <joint name="${prefix}left_finger_tip_joint">
+                        <param name="mimic">${prefix}right_finger_bottom_joint</param>
+                        <param name="multiplier">-1</param>
+                        <xacro:if value="${use_fake_hardware or sim_isaac or sim_gazebo}">
+                            <state_interface name="position"/>
+                            <state_interface name="velocity"/>
+                        </xacro:if>
+                    </joint>
             </xacro:if>
         </ros2_control>

File: kortex_description/grippers/gen3_lite_2f/urdf/gen3_lite_2f_macro.xacro (robot description, xacro)
@@ -139,4 +139,5 @@
         <axis xyz="0 0 1" />
         <limit lower="-0.50" upper="0.21" effort="1000" velocity="1000" /> <!--limit lower="-1.03" upper="0.21" effort="1000" velocity="1000" /-->
+        <mimic joint="${prefix}right_finger_bottom_joint" multiplier="-0.276" offset="-0.1"/>
       </joint>
       <link name="${prefix}left_finger_prox_link">
@@ -172,4 +173,5 @@
         <limit lower="-0.96" upper="0.09" effort="10" velocity="0.6" />
         <dynamics damping="0.1" friction="1"/>
+        <mimic joint="${prefix}right_finger_bottom_joint" multiplier="-1.0" offset="0.0"/>
       </joint>
       <link name="${prefix}left_finger_dist_link">
@@ -204,4 +206,5 @@
         <axis xyz="0 0 -1" />
         <limit lower="-0.50" upper="0.21" effort="1000" velocity="1000" /> <!--limit lower="-1.03" upper="0.21" effort="1000" velocity="1000" /-->
+        <mimic joint="${prefix}right_finger_bottom_joint" multiplier="-0.276" offset="-0.1"/>
       </joint>
     </xacro:unless>
@@ -346,5 +349,5 @@
         <axis xyz="0 0 1" />
         <limit lower="0.0" upper="0.85" effort="1000" velocity="1000" />
-        <mimic joint="${prefix}right_finger_bottom_joint" multiplier="1.0" offset="0.0" />
+        <mimic joint="${prefix}right_finger_bottom_joint" multiplier="-1.0" offset="0.0" />
       </joint>
       <link name="${prefix}left_finger_dist_link">

Commit message: Adjust left finger multiplier

File: kortex_description/grippers/gen3_lite_2f/urdf/gen3_lite_2f.ros2_control.xacro (robot description, xacro)
@@ -70,26 +70,29 @@
                         <param name="mimic">${prefix}right_finger_bottom_joint</param>
                         <param name="multiplier">-1</param>
-                        <xacro:if value="${use_fake_hardware or sim_isaac or sim_gazebo}">
-                            <state_interface name="position"/>
-                            <state_interface name="velocity"/>
-                        </xacro:if>
-                    </joint>
-                    <joint name="${prefix}left_finger_bottom_joint">
-                        <param name="mimic">${prefix}right_finger_bottom_joint</param>
-                        <param name="multiplier">-1</param>
-                        <xacro:if value="${use_fake_hardware or sim_isaac or sim_gazebo}">
-                            <state_interface name="position"/>
-                            <state_interface name="velocity"/>
-                        </xacro:if>
+                        <state_interface name="position"/>
+                        <state_interface name="velocity"/>
                     </joint>
                     <joint name="${prefix}left_finger_tip_joint">
                         <param name="mimic">${prefix}right_finger_bottom_joint</param>
                         <param name="multiplier">-1</param>
-                        <xacro:if value="${use_fake_hardware or sim_isaac or sim_gazebo}">
-                            <state_interface name="position"/>
-                            <state_interface name="velocity"/>
-                        </xacro:if>
+                        <state_interface name="position"/>
+                        <state_interface name="velocity"/>
                     </joint>
             </xacro:if>
+            <!-- The left finger bottom joint exists in both real and simulated setups.
+                 Its multiplier depends on whether we are simulating or running on hardware. -->
+            <joint name="${prefix}left_finger_bottom_joint">
+                <param name="mimic">${prefix}right_finger_bottom_joint</param>
+                <xacro:if value="${use_fake_hardware or sim_isaac or sim_gazebo}">
+                    <param name="multiplier">-1</param>
+                </xacro:if>
+                <xacro:unless value="${use_fake_hardware or sim_isaac or sim_gazebo}">
+                    <param name="multiplier">1</param>
+                </xacro:unless>
+                <xacro:if value="${use_fake_hardware or sim_isaac or sim_gazebo}">
+                    <state_interface name="position"/>
+                    <state_interface name="velocity"/>
+                </xacro:if>
+            </joint>
         </ros2_control>
     </xacro:macro>

Commit message: Update gen3_lite_2f.ros2_control.xacro
The modified file removes the mimic joint definitions and associated <param mimic> and <param multiplier> tags for the gripper's tip and left finger joints. Instead, it conditionally includes only the state interfaces for these joints under use_fake_hardware or sim_isaac, explicitly excluding sim_gazebo. Additionally, the initial position value of the right_finger_bottom_joint state interface was changed from 0.0 to 0.2, and comments were updated to clarify that mimic joints are no longer defined and that Gazebo does not require mimic joint state interfaces. The overall structure is cleaner and more simulation-specific in its conditional logic.

File: kortex_description/grippers/gen3_lite_2f/urdf/gen3_lite_2f.ros2_control.xacro (robot description, xacro)
@@ -53,10 +53,9 @@
                 </xacro:unless>
             </hardware>
-            <!-- Joint interfaces -->
-            <!-- With Gazebo or Hardware, they handle mimic joints, so we only need this command interface activated -->
+            <!-- Always define the commanded joint -->
             <joint name="${prefix}right_finger_bottom_joint">
                 <command_interface name="position" />
                 <state_interface name="position">
-                    <param name="initial_value">0.0</param>
+                    <param name="initial_value">0.2</param>
                 </state_interface>
                 <state_interface name="velocity">
@@ -64,31 +63,18 @@
                 </state_interface>
             </joint>
-            <!-- When simulating we need to include the rest of the gripper joints -->
-            <xacro:if value="${use_fake_hardware or sim_isaac or sim_gazebo}">
-                <!-- Always define mimic joints -->
-                    <joint name="${prefix}right_finger_tip_joint">
-                        <param name="mimic">${prefix}right_finger_bottom_joint</param>
-                        <param name="multiplier">-1</param>
-                        <xacro:if value="${use_fake_hardware or sim_isaac or sim_gazebo}">
-                            <state_interface name="position"/>
-                            <state_interface name="velocity"/>
-                        </xacro:if>
-                    </joint>
-                    <joint name="${prefix}left_finger_bottom_joint">
-                        <param name="mimic">${prefix}right_finger_bottom_joint</param>
-                        <param name="multiplier">-1</param>
-                        <xacro:if value="${use_fake_hardware or sim_isaac or sim_gazebo}">
-                            <state_interface name="position"/>
-                            <state_interface name="velocity"/>
-                        </xacro:if>
-                    </joint>
-                    <joint name="${prefix}left_finger_tip_joint">
-                        <param name="mimic">${prefix}right_finger_bottom_joint</param>
-                        <param name="multiplier">-1</param>
-                        <xacro:if value="${use_fake_hardware or sim_isaac or sim_gazebo}">
-                            <state_interface name="position"/>
-                            <state_interface name="velocity"/>
-                        </xacro:if>
-                    </joint>
+            <!-- In fake hardware or Isaac simulation, define state interfaces for mimics. NOT for Gazebo. -->
+            <xacro:if value="${use_fake_hardware or sim_isaac}">
+                <joint name="${prefix}right_finger_tip_joint">
+                    <state_interface name="position"/>
+                    <state_interface name="velocity"/>
+                </joint>
+                <joint name="${prefix}left_finger_bottom_joint">
+                    <state_interface name="position"/>
+                    <state_interface name="velocity"/>
+                </joint>
+                <joint name="${prefix}left_finger_tip_joint">
+                    <state_interface name="position"/>
+                    <state_interface name="velocity"/>
+                </joint>
             </xacro:if>
         </ros2_control>
