Commit message: Correct the gripper mimic multipliers so the simulated fingers track
With the interface conflict resolved, the simulated gripper still would
not move: goals were accepted and right_finger_bottom_joint stayed at
zero.

The cause was the multipliers on the follower joints. All three were
declared multiplier="-1", but the URDF's <mimic> tags in
gen3_lite_2f_macro.xacro say 1.0 for left_finger_bottom_joint and
-0.276 with offset -0.1 for the two finger tips. gz_ros2_control applies
mimics in software each write() cycle (gz_system.cpp, "set values of all
mimic joints with respect to mimicked joint"), so the wrong multiplier
drove the followers against the URDF and stalled the driven joint.

Match the multiplier/offset pairs to the URDF, and add the offsets, which
were missing entirely.

Verified in headless Gazebo (gz-sim 8.11.0, dartsim, gz_ros2_control
1.2.19) by reading link poses out of the physics engine. Commanding the
gripper from 0.0 to 0.8 rad, per-link change:

                            before              after
  right_finger_prox_link    45.84 deg           45.84 deg
  right_finger_dist_link    38.94 mm            38.94 mm
  left_finger_prox_link      0.00 deg           45.84 deg
  left_finger_dist_link      0.00 mm            38.94 mm

Both fingers now move symmetrically through 45.84 deg, which is the
commanded 0.8 rad. Fingertip separation goes 112.3 mm open to 35.2 mm
closed and back, matching forward kinematics off the URDF to within
0.1 mm; before the change the closed figure was 74.0 mm, the value
predicted when no mimic is applied at all.

Note that gz still logs

  [Err] [Physics.cc:1808] Attempting to create a mimic constraint for
  joint [left_finger_bottom_joint] but the chosen physics engine does not
  support mimic constraints, so no constraint will be created.

That comes from the URDF <mimic> tags during model conversion and is
independent of these declarations. It is not fatal: gz_ros2_control's
software mimic drives the followers regardless, as the measurements
above show.

Co-Authored-By: Claude Opus 5 <noreply@anthropic.com>
Claude-Session: https://claude.ai/code/session_01HPYCorCh7pASi2ipJFeqJb

File: kortex_description/grippers/gen3_lite_2f/urdf/gen3_lite_2f.ros2_control.xacro (robot description, xacro)
@@ -64,9 +64,11 @@
                 </state_interface>
             </joint>
-            <!-- When simulating we need to include the rest of the gripper joints -->
+            <!-- Follower joints. multiplier/offset must match the <mimic>
+                 tags in gen3_lite_2f_macro.xacro. -->
             <xacro:if value="${use_fake_hardware or sim_isaac or sim_gazebo}">
                 <joint name="${prefix}right_finger_tip_joint">
                     <param name="mimic">${prefix}right_finger_bottom_joint</param>
-                    <param name="multiplier">-1</param>
+                    <param name="multiplier">-0.276</param>
+                    <param name="offset">-0.1</param>
                     <xacro:unless value="${sim_gazebo}">
                         <state_interface name="position"/>
@@ -76,5 +78,6 @@
                 <joint name="${prefix}left_finger_bottom_joint">
                     <param name="mimic">${prefix}right_finger_bottom_joint</param>
-                    <param name="multiplier">-1</param>
+                    <param name="multiplier">1.0</param>
+                    <param name="offset">0.0</param>
                     <xacro:unless value="${sim_gazebo}">
                         <state_interface name="position"/>
@@ -84,5 +87,6 @@
                 <joint name="${prefix}left_finger_tip_joint">
                     <param name="mimic">${prefix}right_finger_bottom_joint</param>
-                    <param name="multiplier">-1</param>
+                    <param name="multiplier">-0.276</param>
+                    <param name="offset">-0.1</param>
                     <xacro:unless value="${sim_gazebo}">
                         <state_interface name="position"/>
