Commit message: Give the Gen3 lite gripper joint one owner in Gazebo and load its plugin
Three changes to the Gen3 lite 2F gripper's ros2_control description:

- The gripper system named its Gazebo plugin gz_ros2_control/GzSimSystem,
  a class gz_ros2_control does not export on Jazzy (it exports
  GazeboSimSystem). Gazebo bringup printed "The plugin failed to load"
  and dropped the gripper system on every launch.

- Under Gazebo and Isaac, the arm's system and the gripper's system both
  declared a position command interface on right_finger_bottom_joint.
  The arm's condition was "unless use_fake_hardware"; it is now the exact
  complement of the gripper system's condition, so in every mode one
  system declares the joint. Removes the commented-out remains of an
  earlier attempt at the same guard.

- The follower joints' mimic multipliers were all -1. They now match the
  <mimic> tags in gen3_lite_2f_macro.xacro (1.0 for the left bottom
  joint, -0.276 with offset -0.1 for the two tips), since gz_ros2_control
  applies these in software.

Checked in the course image (kinova-jazzy-20261008) with this and the
FakeSystem change applied: the Lab 6 reference pipeline passed every check
with and without this change, run in isolated containers. Closed-finger
readings on a block were 0.439 to 0.454 with it and 0.428 to 0.452
without; a miss read 0.800 in both. Gazebo bringup logged no errors with
it and the plugin error without it. Expanding the description in each
mode (real, fake, Gazebo) shows each joint declared by one system.

File: kortex_description/grippers/gen3_lite_2f/urdf/gen3_lite_2f.ros2_control.xacro (robot description, xacro)
@@ -30,5 +30,5 @@
                 </xacro:if>
                 <xacro:if value="${sim_gazebo}">
-                    <plugin>gz_ros2_control/GzSimSystem</plugin>
+                    <plugin>gz_ros2_control/GazeboSimSystem</plugin>
                 </xacro:if>
                 <xacro:if value="${use_fake_hardware}">
@@ -64,9 +64,11 @@
                 </state_interface>
             </joint>
-            <!-- When simulating we need to include the rest of the gripper joints -->
+            <!-- Follower joints. multiplier/offset must match the <mimic>
+                 tags in gen3_lite_2f_macro.xacro. -->
             <xacro:if value="${use_fake_hardware or sim_isaac or sim_gazebo}">
                 <joint name="${prefix}right_finger_tip_joint">
                     <param name="mimic">${prefix}right_finger_bottom_joint</param>
-                    <param name="multiplier">-1</param>
+                    <param name="multiplier">-0.276</param>
+                    <param name="offset">-0.1</param>
                     <xacro:unless value="${sim_gazebo}">
                         <state_interface name="position"/>
@@ -76,5 +78,6 @@
                 <joint name="${prefix}left_finger_bottom_joint">
                     <param name="mimic">${prefix}right_finger_bottom_joint</param>
-                    <param name="multiplier">-1</param>
+                    <param name="multiplier">1.0</param>
+                    <param name="offset">0.0</param>
                     <xacro:unless value="${sim_gazebo}">
                         <state_interface name="position"/>
@@ -84,5 +87,6 @@
                 <joint name="${prefix}left_finger_tip_joint">
                     <param name="mimic">${prefix}right_finger_bottom_joint</param>
-                    <param name="multiplier">-1</param>
+                    <param name="multiplier">-0.276</param>
+                    <param name="offset">-0.1</param>
                     <xacro:unless value="${sim_gazebo}">
                         <state_interface name="position"/>
