Commit message: Fix left_finger_bottom_joint mimic direction for real hardware
Changed multiplier from -1.0 to 1.0 under moveit_active block to match real robot behavior. Simulation uses the negative multiplier.

File: kortex_description/grippers/gen3_lite_2f/urdf/gen3_lite_2f_macro.xacro (robot description, xacro)
@@ -349,5 +349,5 @@
         <axis xyz="0 0 1" />
         <limit lower="0.0" upper="0.85" effort="1000" velocity="1000" />
-        <mimic joint="${prefix}right_finger_bottom_joint" multiplier="-1.0" offset="0.0" />
+        <mimic joint="${prefix}right_finger_bottom_joint" multiplier="1.0" offset="0.0" />
       </joint>
       <link name="${prefix}left_finger_dist_link">

Commit message: Update gen3_lite_2f_macro.xacro. Refined gripper mimic behavior and joint parameters
The updated file introduces multiple structural and numerical changes across hardware configurations, improving consistency and simulation support. Key modifications include corrected mimic joint parameters for the right_finger_tip_joint and left_finger_tip_joint within the simulated path

File: kortex_description/grippers/gen3_lite_2f/urdf/gen3_lite_2f_macro.xacro (robot description, xacro)
@@ -108,37 +108,37 @@
         <dynamics damping="0.1" friction="1"/>
       </joint>
-      <link name="${prefix}right_finger_dist_link">
-        <inertial>
-          <origin xyz="0.018488 0.0011091 0" rpy="0 0 0" />
-          <mass value="0.010748" />
-          <inertia ixx="6.3E-07" ixy="3.2E-07" ixz="0" iyy="1.83E-06" iyz="0" izz="1.61E-06" />
-        </inertial>
-        <visual>
-          <origin xyz="0 0 0" rpy="0 0 0" />
-          <geometry>
-            <mesh filename="file://$(find kortex_description)/grippers/gen3_lite_2f/meshes/right_finger_dist_link.STL" />
-          </geometry>
-          <material name="">
-            <color rgba="0 0.055 0.525 1" />
-          </material>
-        </visual>
-        <collision>
-          <origin xyz="0 0 0" rpy="0 0 0" />
-          <geometry>
-            <mesh filename="file://$(find kortex_description)/grippers/gen3_lite_2f/meshes/right_finger_dist_link.STL" />
-          </geometry>
-        </collision>
-      </link>
-      <gazebo reference="${prefix}right_finger_dist_link">
-        <material>Kortex/Blue</material>
-      </gazebo>
-      <joint name="${prefix}right_finger_tip_joint" type="revolute">
-        <origin xyz="-0.045636 0.020423 0" rpy="0 0 0" />
-        <parent link="${prefix}right_finger_prox_link" />
-        <child link="${prefix}right_finger_dist_link" />
-        <axis xyz="0 0 1" />
-        <limit lower="-0.50" upper="0.21" effort="1000" velocity="1000" /> <!--limit lower="-1.03" upper="0.21" effort="1000" velocity="1000" /-->
-        <mimic joint="${prefix}right_finger_bottom_joint" multiplier="-0.276" offset="-0.1"/>
-      </joint>
+    <link name="right_finger_dist_link">
+      <inertial>
+        <origin xyz="0.018488 0.0011091 0" rpy="0 0 0" />
+        <mass value="0.010748" />
+        <inertia ixx="6.3E-07" ixy="3.2E-07" ixz="0" iyy="1.83E-06" iyz="0" izz="1.61E-06" />
+      </inertial>
+      <visual>
+        <origin xyz="0 0 0" rpy="0 0 0" />
+        <geometry>
+          <mesh filename="package://kortex_description/grippers/gen3_lite_2f/meshes/right_finger_dist_link.STL" />
+        </geometry>
+        <material name="">
+          <color rgba="0 0.055 0.525 1" />
+        </material>
+      </visual>
+      <collision>
+        <origin xyz="0 0 0" rpy="0 0 0" />
+        <geometry>
+          <mesh filename="package://kortex_description/grippers/gen3_lite_2f/meshes/right_finger_dist_link.STL" />
+        </geometry>
+      </collision>
+    </link>
+    <gazebo reference="right_finger_dist_link">
+      <material>Kortex/Blue</material>
+    </gazebo>
+    <joint name="right_finger_tip_joint" type="revolute">
+      <origin xyz="-0.045636 0.020423 6.9901E-05" rpy="0 0 0" />
+      <parent link="right_finger_prox_link" />
+      <child link="right_finger_dist_link" />
+      <axis xyz="0 0 1" />
+      <limit lower="-0.50" upper="0.21" effort="1000" velocity="1000" /> <!--limit lower="-1.03" upper="0.21" effort="1000" velocity="1000" /-->
+      <mimic joint="right_finger_bottom_joint" multiplier="-0.676" offset="0.149"/>
+    </joint>
       <link name="${prefix}left_finger_prox_link">
         <inertial>
@@ -173,5 +173,5 @@
         <limit lower="-0.96" upper="0.09" effort="10" velocity="0.6" />
         <dynamics damping="0.1" friction="1"/>
-        <mimic joint="${prefix}right_finger_bottom_joint" multiplier="-1.0" offset="0.0"/>
+        <mimic joint="right_finger_bottom_joint" multiplier="-1" offset="0.0" />
       </joint>
       <link name="${prefix}left_finger_dist_link">
@@ -206,5 +206,5 @@
         <axis xyz="0 0 -1" />
         <limit lower="-0.50" upper="0.21" effort="1000" velocity="1000" /> <!--limit lower="-1.03" upper="0.21" effort="1000" velocity="1000" /-->
-        <mimic joint="${prefix}right_finger_bottom_joint" multiplier="-0.276" offset="-0.1"/>
+        <mimic joint="right_finger_bottom_joint" multiplier="-0.676" offset="0.149" />
       </joint>
     </xacro:unless>

Commit message: Update gen3_lite_2f_macro.xacro real robot values to match simulation
Synchronized the real robot joint parameters with simulation values:
- right_finger_bottom_joint: updated origin rpy, axis, limits, added dynamics
- left_finger_bottom_joint: updated origin rpy, limits, mimic multiplier, added dynamics
- right/left_finger_tip_joint: updated mimic multiplier/offset values

https://claude.ai/code/session_01AUyHjfRyHkJzrqMTF2Vh15

File: kortex_description/grippers/gen3_lite_2f/urdf/gen3_lite_2f_macro.xacro (robot description, xacro)
@@ -277,11 +277,11 @@
         <material>Kortex/Gray</material>
       </gazebo>
-      <!-- TODO(MarqRazz) look into why the joint and limits needed to be flipped and modified -->
       <joint name="${prefix}right_finger_bottom_joint" type="revolute">
-        <origin xyz="0 -0.030501 0.070003" rpy="1.571 0.611 1.571" />
+        <origin xyz="0 -0.030501 0.070003" rpy="0 1.5708 0" />
         <parent link="${prefix}gripper_base_link" />
         <child link="${prefix}right_finger_prox_link" />
-        <axis xyz="0 0 -1" />
-        <limit lower="0.0" upper="0.85" effort="50" velocity="0.6" />
+        <axis xyz="0 0 1" />
+        <limit lower="-0.09" upper="0.96" effort="10" velocity="0.6" />
+        <dynamics damping="0.1" friction="1"/>
       </joint>
       <link name="${prefix}right_finger_dist_link">
@@ -311,10 +311,10 @@
       </gazebo>
       <joint name="${prefix}right_finger_tip_joint" type="revolute">
-        <origin xyz="-0.045636 0.020423 0" rpy="0 0 0" />
+        <origin xyz="-0.045636 0.020423 6.9901E-05" rpy="0 0 0" />
         <parent link="${prefix}right_finger_prox_link" />
         <child link="${prefix}right_finger_dist_link" />
         <axis xyz="0 0 1" />
         <limit lower="-0.50" upper="0.21" effort="1000" velocity="1000" /> <!--limit lower="-1.03" upper="0.21" effort="1000" velocity="1000" /-->
-        <mimic joint="${prefix}right_finger_bottom_joint" multiplier="-0.276" offset="-0.1" />
+        <mimic joint="${prefix}right_finger_bottom_joint" multiplier="-0.676" offset="0.149" />
       </joint>
       <link name="${prefix}left_finger_prox_link">
@@ -344,10 +344,11 @@
       </gazebo>
       <joint name="${prefix}left_finger_bottom_joint" type="revolute">
-        <origin xyz="0 0.0305 0.070003" rpy="-1.571 0.611 -1.571" />
+        <origin xyz="0 0.0305 0.070003" rpy="0 1.5708 0" />
         <parent link="${prefix}gripper_base_link" />
         <child link="${prefix}left_finger_prox_link" />
         <axis xyz="0 0 1" />
-        <limit lower="0.0" upper="0.85" effort="1000" velocity="1000" />
-        <mimic joint="${prefix}right_finger_bottom_joint" multiplier="1.0" offset="0.0" />
+        <limit lower="-0.96" upper="0.09" effort="10" velocity="0.6" />
+        <dynamics damping="0.1" friction="1"/>
+        <mimic joint="${prefix}right_finger_bottom_joint" multiplier="-1" offset="0.0" />
       </joint>
       <link name="${prefix}left_finger_dist_link">
@@ -382,5 +383,5 @@
         <axis xyz="0 0 -1" />
         <limit lower="-0.50" upper="0.21" effort="1000" velocity="1000" /> <!--limit lower="-1.03" upper="0.21" effort="1000" velocity="1000" /-->
-        <mimic joint="${prefix}right_finger_bottom_joint" multiplier="-0.276" offset="-0.1" />
+        <mimic joint="${prefix}right_finger_bottom_joint" multiplier="-0.676" offset="0.149" />
       </joint>
     </xacro:unless>
