Commit message: Align the moveit_active gripper block with the real-hardware kinematics
gen3_lite_2f_macro.xacro defines the gripper three times: once for
sim (use_fake_hardware/sim_gazebo/sim_isaac), once for real hardware, and
once under moveit_active. The gen3_lite MoveIt fixes rewrote the first two
blocks but left the moveit_active block on the pre-fix geometry, so
right_finger_bottom_joint ended up with axis "0 0 1" there against
"0 0 -1" everywhere else.

Because sim.launch.py declares moveit_active with default_value "true"
while robot.launch.py never passes it (falling back to the xacro default
of false), simulation rendered the moveit_active block and real hardware
rendered the real-hardware block. The same commanded gripper position
therefore rotated the fingers in opposite directions -- commanding a
close in sim opened the gripper on the arm and vice versa.

Bring the moveit_active block's four finger joints in line with the
real-hardware block: flip right_finger_bottom_joint's axis, use the
re-derived finger origins, drop left_finger_bottom_joint's inverted
mimic in favour of the 1.0 multiplier, and use the -0.276/-0.1 finger
tip mimics.

Co-Authored-By: Claude Opus 5 <noreply@anthropic.com>
Claude-Session: https://claude.ai/code/session_01HPYCorCh7pASi2ipJFeqJb

File: kortex_description/grippers/gen3_lite_2f/urdf/gen3_lite_2f_macro.xacro (robot description, xacro)
@@ -453,9 +453,9 @@
     </gazebo>
     <joint name="right_finger_bottom_joint" type="revolute">
-      <origin xyz="0 -0.030501 0.070003" rpy="0 1.5708 0" />
+      <origin xyz="0 -0.030501 0.070003" rpy="1.571 0.611 1.571" />
       <parent link="gripper_base_link" />
       <child link="right_finger_prox_link" />
-      <axis xyz="0 0 1" />
-      <limit lower="0.0" upper="0.96" effort="1000" velocity="0.6" />
+      <axis xyz="0 0 -1" />
+      <limit lower="0.0" upper="0.85" effort="1000" velocity="0.6" />
     </joint>
     <link name="right_finger_dist_link">
@@ -490,5 +490,5 @@
       <axis xyz="0 0 1" />
       <limit lower="-0.50" upper="0.21" effort="1000" velocity="1000" /> <!--limit lower="-1.03" upper="0.21" effort="1000" velocity="1000" /-->
-      <mimic joint="right_finger_bottom_joint" multiplier="-0.676" offset="0.149" />
+      <mimic joint="right_finger_bottom_joint" multiplier="-0.276" offset="-0.1" />
     </joint>
     <link name="left_finger_prox_link">
@@ -518,10 +518,10 @@
     </gazebo>
     <joint name="left_finger_bottom_joint" type="revolute">
-      <origin xyz="0 0.0305 0.070003" rpy="0 1.5708 0" />
+      <origin xyz="0 0.0305 0.070003" rpy="-1.571 0.611 -1.571" />
       <parent link="gripper_base_link" />
       <child link="left_finger_prox_link" />
       <axis xyz="0 0 1" />
-      <limit lower="-0.96" upper="0.0" effort="1000" velocity="1000" />
-      <mimic joint="right_finger_bottom_joint" multiplier="-1.0" offset="0.0" />
+      <limit lower="0.0" upper="0.85" effort="1000" velocity="1000" />
+      <mimic joint="right_finger_bottom_joint" multiplier="1.0" offset="0.0" />
     </joint>
     <link name="left_finger_dist_link">
@@ -556,5 +556,5 @@
       <axis xyz="0 0 -1" />
       <limit lower="-0.50" upper="0.21" effort="1000" velocity="1000" /> <!--limit lower="-1.03" upper="0.21" effort="1000" velocity="1000" /-->
-      <mimic joint="right_finger_bottom_joint" multiplier="-0.676" offset="0.149" />
+      <mimic joint="right_finger_bottom_joint" multiplier="-0.276" offset="-0.1" />
     </joint>
   </xacro:if>
