Commit message: Declare the Gen3 lite 2F gripper geometry once instead of three times
The gripper description was written out three times in full -- once under
"use_fake_hardware or sim_isaac or sim_gazebo", once for real hardware,
and once under moveit_active -- because the three modes need different
ros2_control tags. Duplicating the whole kinematic chain to vary the
control tags is what let the three copies drift apart, and the
moveit_active copy had been left behind entirely: it still carried the
pre-fix joint axes, and it hardcoded link and joint names with no
${prefix} at all.

The arm macro next door already solves the same problem the right way, by
defining its joints once and letting moveit_active select only a
property, so follow that pattern here. The geometry is now declared a
single time and the values that genuinely vary per mode are hoisted into
properties, each mode keeping the numbers it had:

                     sim      real     moveit_active
  finger limits   -0.1/0.96  0.0/0.85    0.0/0.85
  right effort       10         50         1000
  left effort        10        1000        1000
  left velocity      0.6       1000        1000
  <dynamics>         yes        no          no

Verified by expanding gen3_lite_gen3_lite_2f.xacro before and after in
every mode (real, moveit_active, sim_gazebo, use_fake_hardware,
sim_isaac, gazebo+moveit, and prefixed): the generated URDFs are
identical apart from the two intentional changes below.

Two intentional changes:

- Mesh URIs move from file://$(find kortex_description) to package://.
  Every other description in the package already uses package://; the
  two non-moveit blocks here were the last 20 file:// references in the
  tree, and the moveit_active block was already on package://.

- The stale "TODO(MarqRazz) look into why the joint and limits needed to
  be flipped and modified" comment is dropped, since there is now one
  definition and nothing left to reconcile.

Because the geometry is shared, prefix now applies in the moveit_active
case too. Previously "prefix:=arm1_ moveit_active:=true" emitted a URDF
whose ros2_control block drove arm1_right_finger_bottom_joint while the
gripper only defined the unprefixed right_finger_bottom_joint, along with
two joints parented to a nonexistent dummy_link.

Co-Authored-By: Claude Opus 5 <noreply@anthropic.com>
Claude-Session: https://claude.ai/code/session_01HPYCorCh7pASi2ipJFeqJb

File: kortex_description/grippers/gen3_lite_2f/urdf/gen3_lite_2f_macro.xacro (robot description, xacro)
@@ -13,419 +13,78 @@
     use_internal_bus_gripper_comm:=true
     moveit_active:=false">
-  <xacro:if value="${use_fake_hardware or sim_isaac or sim_gazebo}">
-    <xacro:unless value="${moveit_active}">
+  <!-- The gripper only needs a ros2_control system of its own when it is being
+       simulated and is not driven through MoveIt. On real hardware the arm's
+       KortexMultiInterfaceHardware already exposes the gripper over the
+       internal bus, and the moveit_active description is control-free by
+       design. -->
+  <xacro:property name="simulated" value="${(use_fake_hardware or sim_isaac or sim_gazebo) and not moveit_active}"/>
+  <!-- Per-mode finger tuning.
+       This description used to be written out three times over (once for
+       simulation, once for real hardware, once for moveit_active) and the
+       copies had drifted apart: they disagreed not only on the values below
+       but, until recently, on the joint axes and mimic multipliers as well,
+       which meant the same gripper command opened the fingers in one mode and
+       closed them in another. The geometry is now declared exactly once and
+       only the values that genuinely vary are parameterised here, each mode
+       keeping the numbers it already had. -->
+  <xacro:property name="finger_lower" value="${-0.1 if simulated else 0.0}"/>
+  <xacro:property name="finger_upper" value="${0.96 if simulated else 0.85}"/>
+  <xacro:property name="right_bottom_effort" value="${10 if simulated else (1000 if moveit_active else 50)}"/>
+  <xacro:property name="left_bottom_effort" value="${10 if simulated else 1000}"/>
+  <xacro:property name="left_bottom_velocity" value="${0.6 if simulated else 1000}"/>
+  <xacro:if value="${simulated}">
     <!-- ros2 control include -->
-      <xacro:include filename="$(find kortex_description)/grippers/gen3_lite_2f/urdf/gen3_lite_2f.ros2_control.xacro" />
-      <xacro:if value="${sim_gazebo}">
-        <xacro:property name="ros2_control_name" value="GazeboSimSystem"/>
-      </xacro:if>
-      <xacro:if value="${use_fake_hardware}">
-        <xacro:property name="ros2_control_name" value="GenericSystem"/>
-      </xacro:if>
-      <xacro:unless value="${use_fake_hardware or sim_gazebo}">
-        <xacro:property name="ros2_control_name" value="${prefix}KortexMultiInterfaceHardware"/>
-      </xacro:unless>
-      <xacro:gripper_ros2_control
-        prefix="${prefix}"
-        use_fake_hardware="${use_fake_hardware}"
-        fake_sensor_commands="${fake_sensor_commands}"
-        sim_gazebo="${sim_gazebo}"
-        sim_isaac="${sim_isaac}"
-        isaac_joint_commands="${isaac_joint_commands}"
-        isaac_joint_states="${isaac_joint_states}"
-        tf_prefix=""/>
+    <xacro:include filename="$(find kortex_description)/grippers/gen3_lite_2f/urdf/gen3_lite_2f.ros2_control.xacro" />
+    <xacro:gripper_ros2_control
+      prefix="${prefix}"
+      use_fake_hardware="${use_fake_hardware}"
+      fake_sensor_commands="${fake_sensor_commands}"
+      sim_gazebo="${sim_gazebo}"
+      sim_isaac="${sim_isaac}"
+      isaac_joint_commands="${isaac_joint_commands}"
+      isaac_joint_states="${isaac_joint_states}"
+      tf_prefix=""/>
+  </xacro:if>
   <!-- Tool frame used by the arm -->
-      <link name="${prefix}tool_frame"/>
-      <joint name="${prefix}tool_frame_joint" type="fixed">
-          <origin xyz="0 0 0.130" rpy="0 0 1.57079632679" />
-          <parent link="${parent}" />
-          <child link="${prefix}tool_frame" />
-          <axis xyz="0 0 0" />
-      </joint>
-      <!-- Gripper description -->
-      <joint name="${prefix}gripper_base_joint" type="fixed">
-        <origin xyz="0 0 0" rpy="0 0 0" />
-        <parent link="${parent}" />
-        <child link="${prefix}gripper_base_link" />
-        <axis xyz="0 0 0" />
-      </joint>
-      <link name="${prefix}gripper_base_link">
-        <inertial>
-          <origin xyz="4.03E-06 1.08E-05 0.041397" rpy="0 0 0" />
-          <mass value="0.1395" />
-          <inertia ixx="0.00011614" ixy="1E-08" ixz="4E-08" iyy="0.00010327" iyz="0" izz="9.707E-05" />
-        </inertial>
-        <visual>
-          <origin xyz="0 0 0" rpy="0 0 0" />
-          <geometry>
-            <mesh filename="file://$(find kortex_description)/grippers/gen3_lite_2f/meshes/gripper_base_link.STL" />
-          </geometry>
-          <material name="">
-            <color rgba="0.803 0.824 0.820 1" />
-          </material>
-        </visual>
-        <collision>
-          <origin xyz="0 0 0" rpy="0 0 0" />
-          <geometry>
-            <mesh filename="file://$(find kortex_description)/grippers/gen3_lite_2f/meshes/gripper_base_link.STL" />
-          </geometry>
-        </collision>
-      </link>
-      <gazebo reference="${prefix}gripper_base_link">
-        <material>Kortex/Gray</material>
-      </gazebo>
-      <link name="${prefix}right_finger_prox_link">
-      <inertial>
-        <origin xyz="0.020257 0.0063483 6.991E-05" rpy="0 0 0" />
-        <mass value="0.018385" />
-        <inertia ixx="2.29E-06" ixy="1.43E-06" ixz="0" iyy="4.56E-06" iyz="0" izz="4.77E-06" />
-      </inertial>
-      <visual>
-        <origin xyz="0 0 0" rpy="0 0 0" />
-        <geometry>
-          <mesh filename="file://$(find kortex_description)/grippers/gen3_lite_2f/meshes/right_finger_prox_link.STL" />
-        </geometry>
-        <material name="">
-            <color rgba="0.803 0.824 0.820 1" />
-        </material>
-      </visual>
-      <collision>
-        <origin xyz="0 0 0" rpy="0 0 0" />
-        <geometry>
-          <mesh filename="file://$(find kortex_description)/grippers/gen3_lite_2f/meshes/right_finger_prox_link.STL" />
-        </geometry>
-      </collision>
-      </link>
-      <gazebo reference="${prefix}right_finger_prox_link">
-        <material>Kortex/Gray</material>
-      </gazebo>
-      <joint name="${prefix}right_finger_bottom_joint" type="revolute">
-        <origin xyz="0 -0.030501 0.070003" rpy="1.571 0.611 1.571" />
-        <parent link="${prefix}gripper_base_link" />
-        <child link="${prefix}right_finger_prox_link" />
-        <axis xyz="0 0 -1" />
-        <limit lower="-0.1" upper="0.96" effort="10" velocity="0.6" />
-        <dynamics damping="0.1" friction="1"/>
-      </joint>
-      <link name="${prefix}right_finger_dist_link">
-        <inertial>
-          <origin xyz="0.018488 0.0011091 0" rpy="0 0 0" />
-          <mass value="0.010748" />
-          <inertia ixx="6.3E-07" ixy="3.2E-07" ixz="0" iyy="1.83E-06" iyz="0" izz="1.61E-06" />
-        </inertial>
-        <visual>
-          <origin xyz="0 0 0" rpy="0 0 0" />
-          <geometry>
-            <mesh filename="file://$(find kortex_description)/grippers/gen3_lite_2f/meshes/right_finger_dist_link.STL" />
-          </geometry>
-          <material name="">
-            <color rgba="0 0.055 0.525 1" />
-          </material>
-        </visual>
-        <collision>
-          <origin xyz="0 0 0" rpy="0 0 0" />
-          <geometry>
-            <mesh filename="file://$(find kortex_description)/grippers/gen3_lite_2f/meshes/right_finger_dist_link.STL" />
-          </geometry>
-        </collision>
-      </link>
-      <gazebo reference="${prefix}right_finger_dist_link">
-        <material>Kortex/Blue</material>
-      </gazebo>
-      <joint name="${prefix}right_finger_tip_joint" type="revolute">
-        <origin xyz="-0.045636 0.020423 0" rpy="0 0 0" />
-        <parent link="${prefix}right_finger_prox_link" />
-        <child link="${prefix}right_finger_dist_link" />
-        <axis xyz="0 0 1" />
-        <limit lower="-0.50" upper="0.21" effort="1000" velocity="1000" /> <!--limit lower="-1.03" upper="0.21" effort="1000" velocity="1000" /-->
-        <mimic joint="${prefix}right_finger_bottom_joint" multiplier="-0.276" offset="-0.1" />
-      </joint>
-      <link name="${prefix}left_finger_prox_link">
-        <inertial>
-          <origin xyz="0.020257 0.0063483 6.99E-05" rpy="0 0 0" />
-          <mass value="0.018385" />
-          <inertia ixx="2.29E-06" ixy="1.43E-06" ixz="0" iyy="4.56E-06" iyz="0" izz="4.77E-06" />
-        </inertial>
-        <visual>
-          <origin xyz="0 0 0" rpy="0 0 0" />
-          <geometry>
-            <mesh filename="file://$(find kortex_description)/grippers/gen3_lite_2f/meshes/left_finger_prox_link.STL" />
-          </geometry>
-          <material name="">
-            <color rgba="0.803 0.824 0.820 1" />
-          </material>
-        </visual>
-        <collision>
-          <origin xyz="0 0 0" rpy="0 0 0" />
-          <geometry>
-            <mesh filename="file://$(find kortex_description)/grippers/gen3_lite_2f/meshes/left_finger_prox_link.STL" />
-          </geometry>
-        </collision>
-      </link>
-      <gazebo reference="${prefix}left_finger_prox_link">
-        <material>Kortex/Gray</material>
-      </gazebo>
-      <joint name="${prefix}left_finger_bottom_joint" type="revolute">
-        <origin xyz="0 0.0305 0.070003" rpy="-1.571 0.611 -1.571" />
-        <parent link="${prefix}gripper_base_link" />
-        <child link="${prefix}left_finger_prox_link" />
-        <axis xyz="0 0 1" />
-        <limit lower="-0.1" upper="0.96" effort="10" velocity="0.6" />
-        <dynamics damping="0.1" friction="1"/>
-        <mimic joint="${prefix}right_finger_bottom_joint" multiplier="1.0" offset="0.0" />
-      </joint>
-      <link name="${prefix}left_finger_dist_link">
-        <inertial>
-          <origin xyz="-0.018488 0.0011091 0" rpy="0 0 0" />
-          <mass value="0.010748" />
-          <inertia ixx="6.3E-07" ixy="3.2E-07" ixz="0" iyy="1.83E-06" iyz="0" izz="1.61E-06" />
-        </inertial>
-        <visual>
-          <origin xyz="0 0 0" rpy="0 0 0" />
-          <geometry>
-            <mesh filename="file://$(find kortex_description)/grippers/gen3_lite_2f/meshes/left_finger_dist_link.STL" />
-          </geometry>
-          <material name="">
-            <color rgba="0 0.055 0.525 1" />
-          </material>
-        </visual>
-        <collision>
-          <origin xyz="0 0 0" rpy="0 0 0" />
-          <geometry>
-            <mesh filename="file://$(find kortex_description)/grippers/gen3_lite_2f/meshes/left_finger_dist_link.STL" />
-          </geometry>
-        </collision>
-      </link>
-      <gazebo reference="${prefix}left_finger_dist_link">
-        <material>Kortex/Blue</material>
-      </gazebo>
-      <joint name="${prefix}left_finger_tip_joint" type="revolute">
-        <origin xyz="-0.045636 -0.020423 6.9901E-05" rpy="0 0 0" />
-        <parent link="${prefix}left_finger_prox_link" />
-        <child link="${prefix}left_finger_dist_link" />
-        <axis xyz="0 0 -1" />
-        <limit lower="-0.50" upper="0.21" effort="1000" velocity="1000" /> <!--limit lower="-1.03" upper="0.21" effort="1000" velocity="1000" /-->
-        <mimic joint="${prefix}right_finger_bottom_joint" multiplier="-0.276" offset="-0.1" />
-      </joint>
-    </xacro:unless>
-  </xacro:if>
-  <xacro:unless value="${use_fake_hardware or sim_isaac or sim_gazebo}">
-    <xacro:unless value="${moveit_active}">
-        <!-- Tool frame used by the arm -->
-      <link name="${prefix}tool_frame"/>
-      <joint name="${prefix}tool_frame_joint" type="fixed">
-          <origin xyz="0 0 0.130" rpy="0 0 1.57079632679" />
-          <parent link="${parent}" />
-          <child link="${prefix}tool_frame" />
-          <axis xyz="0 0 0" />
-      </joint>
-      <!-- Gripper description -->
-      <joint name="${prefix}gripper_base_joint" type="fixed">
-        <origin xyz="0 0 0" rpy="0 0 0" />
-        <parent link="${parent}" />
-        <child link="${prefix}gripper_base_link" />
-        <axis xyz="0 0 0" />
-      </joint>
-      <link name="${prefix}gripper_base_link">
-        <inertial>
-          <origin xyz="4.03E-06 1.08E-05 0.041397" rpy="0 0 0" />
-          <mass value="0.1395" />
-          <inertia ixx="0.00011614" ixy="1E-08" ixz="4E-08" iyy="0.00010327" iyz="0" izz="9.707E-05" />
-        </inertial>
-        <visual>
-          <origin xyz="0 0 0" rpy="0 0 0" />
-          <geometry>
-            <mesh filename="file://$(find kortex_description)/grippers/gen3_lite_2f/meshes/gripper_base_link.STL" />
-          </geometry>
-          <material name="">
-            <color rgba="0.803 0.824 0.820 1" />
-          </material>
-        </visual>
-        <collision>
-          <origin xyz="0 0 0" rpy="0 0 0" />
-          <geometry>
-            <mesh filename="file://$(find kortex_description)/grippers/gen3_lite_2f/meshes/gripper_base_link.STL" />
-          </geometry>
-        </collision>
-      </link>
-      <gazebo reference="${prefix}gripper_base_link">
-        <material>Kortex/Gray</material>
-      </gazebo>
-      <link name="${prefix}right_finger_prox_link">
-      <inertial>
-        <origin xyz="0.020257 0.0063483 6.991E-05" rpy="0 0 0" />
-        <mass value="0.018385" />
-        <inertia ixx="2.29E-06" ixy="1.43E-06" ixz="0" iyy="4.56E-06" iyz="0" izz="4.77E-06" />
-      </inertial>
-      <visual>
-        <origin xyz="0 0 0" rpy="0 0 0" />
-        <geometry>
-          <mesh filename="file://$(find kortex_description)/grippers/gen3_lite_2f/meshes/right_finger_prox_link.STL" />
-        </geometry>
-        <material name="">
-            <color rgba="0.803 0.824 0.820 1" />
-        </material>
-      </visual>
-      <collision>
-        <origin xyz="0 0 0" rpy="0 0 0" />
-        <geometry>
-          <mesh filename="file://$(find kortex_description)/grippers/gen3_lite_2f/meshes/right_finger_prox_link.STL" />
-        </geometry>
-      </collision>
-      </link>
-      <gazebo reference="${prefix}right_finger_prox_link">
-        <material>Kortex/Gray</material>
-      </gazebo>
-      <!-- TODO(MarqRazz) look into why the joint and limits needed to be flipped and modified -->
-      <joint name="${prefix}right_finger_bottom_joint" type="revolute">
-        <origin xyz="0 -0.030501 0.070003" rpy="1.571 0.611 1.571" />
-        <parent link="${prefix}gripper_base_link" />
-        <child link="${prefix}right_finger_prox_link" />
-        <axis xyz="0 0 -1" />
-        <limit lower="0.0" upper="0.85" effort="50" velocity="0.6" />
-      </joint>
-      <link name="${prefix}right_finger_dist_link">
-        <inertial>
-          <origin xyz="0.018488 0.0011091 0" rpy="0 0 0" />
-          <mass value="0.010748" />
-          <inertia ixx="6.3E-07" ixy="3.2E-07" ixz="0" iyy="1.83E-06" iyz="0" izz="1.61E-06" />
-        </inertial>
-        <visual>
-          <origin xyz="0 0 0" rpy="0 0 0" />
-          <geometry>
-            <mesh filename="file://$(find kortex_description)/grippers/gen3_lite_2f/meshes/right_finger_dist_link.STL" />
-          </geometry>
-          <material name="">
-            <color rgba="0 0.055 0.525 1" />
-          </material>
-        </visual>
-        <collision>
-          <origin xyz="0 0 0" rpy="0 0 0" />
-          <geometry>
-            <mesh filename="file://$(find kortex_description)/grippers/gen3_lite_2f/meshes/right_finger_dist_link.STL" />
-          </geometry>
-        </collision>
-      </link>
-      <gazebo reference="${prefix}right_finger_dist_link">
-        <material>Kortex/Blue</material>
-      </gazebo>
-      <joint name="${prefix}right_finger_tip_joint" type="revolute">
-        <origin xyz="-0.045636 0.020423 0" rpy="0 0 0" />
-        <parent link="${prefix}right_finger_prox_link" />
-        <child link="${prefix}right_finger_dist_link" />
-        <axis xyz="0 0 1" />
-        <limit lower="-0.50" upper="0.21" effort="1000" velocity="1000" /> <!--limit lower="-1.03" upper="0.21" effort="1000" velocity="1000" /-->
-        <mimic joint="${prefix}right_finger_bottom_joint" multiplier="-0.276" offset="-0.1" />
-      </joint>
-      <link name="${prefix}left_finger_prox_link">
-        <inertial>
-          <origin xyz="0.020257 0.0063483 6.99E-05" rpy="0 0 0" />
-          <mass value="0.018385" />
-          <inertia ixx="2.29E-06" ixy="1.43E-06" ixz="0" iyy="4.56E-06" iyz="0" izz="4.77E-06" />
-        </inertial>
-        <visual>
-          <origin xyz="0 0 0" rpy="0 0 0" />
-          <geometry>
-            <mesh filename="file://$(find kortex_description)/grippers/gen3_lite_2f/meshes/left_finger_prox_link.STL" />
-          </geometry>
-          <material name="">
-            <color rgba="0.803 0.824 0.820 1" />
-          </material>
-        </visual>
-        <collision>
-          <origin xyz="0 0 0" rpy="0 0 0" />
-          <geometry>
-            <mesh filename="file://$(find kortex_description)/grippers/gen3_lite_2f/meshes/left_finger_prox_link.STL" />
-          </geometry>
-        </collision>
-      </link>
-      <gazebo reference="${prefix}left_finger_prox_link">
-        <material>Kortex/Gray</material>
-      </gazebo>
-      <joint name="${prefix}left_finger_bottom_joint" type="revolute">
-        <origin xyz="0 0.0305 0.070003" rpy="-1.571 0.611 -1.571" />
-        <parent link="${prefix}gripper_base_link" />
-        <child link="${prefix}left_finger_prox_link" />
-        <axis xyz="0 0 1" />
-        <limit lower="0.0" upper="0.85" effort="1000" velocity="1000" />
-        <mimic joint="${prefix}right_finger_bottom_joint" multiplier="1.0" offset="0.0" />
-      </joint>
-      <link name="${prefix}left_finger_dist_link">
-        <inertial>
-          <origin xyz="-0.018488 0.0011091 0" rpy="0 0 0" />
-          <mass value="0.010748" />
-          <inertia ixx="6.3E-07" ixy="3.2E-07" ixz="0" iyy="1.83E-06" iyz="0" izz="1.61E-06" />
-        </inertial>
-        <visual>
-          <origin xyz="0 0 0" rpy="0 0 0" />
-          <geometry>
-            <mesh filename="file://$(find kortex_description)/grippers/gen3_lite_2f/meshes/left_finger_dist_link.STL" />
-          </geometry>
-          <material name="">
-            <color rgba="0 0.055 0.525 1" />
-          </material>
-        </visual>
-        <collision>
-          <origin xyz="0 0 0" rpy="0 0 0" />
-          <geometry>
-            <mesh filename="file://$(find kortex_description)/grippers/gen3_lite_2f/meshes/left_finger_dist_link.STL" />
-          </geometry>
-        </collision>
-      </link>
-      <gazebo reference="${prefix}left_finger_dist_link">
-        <material>Kortex/Blue</material>
-      </gazebo>
-      <joint name="${prefix}left_finger_tip_joint" type="revolute">
-        <origin xyz="-0.045636 -0.020423 6.9901E-05" rpy="0 0 0" />
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