Commit message: Stop the arm and gripper both claiming right_finger_bottom_joint
Under Gazebo and Isaac, two ros2_control systems declared a position
command interface for the same gripper joint: the arm's system in
kortex.ros2_control.xacro, and the gripper's own GripperHardwareInterface
in gen3_lite_2f.ros2_control.xacro. The resource manager rejects the
duplicate and drops the entire gripper system:

  [ERROR] [controller_manager]: Exception of type : St13runtime_error
  occurred while importing command interfaces for the hardware
  'GripperHardwareInterface' : ResourceStorage: Tried to insert
  CommandInterface with already existing key.
  Insert[right_finger_bottom_joint/position]

The gripper system is where the finger mimic parameters are declared, so
losing it means the simulated gripper has no mimic handling at all -- the
driven joint is left exposed by the arm's system with the three follower
joints unlinked.

The arm's condition was "unless use_fake_hardware", which excluded only
the mock-hardware case and overlapped with the gripper on sim_gazebo and
sim_isaac. Make it the exact complement of the gripper's own condition
instead, so the two can never both declare the joint:

  gripper system: (use_fake_hardware or sim_isaac or sim_gazebo) and not moveit_active
  arm system:     the negation of the above

Verified by expanding gen3_lite_gen3_lite_2f.xacro in every mode (real,
moveit_active, sim_gazebo, use_fake_hardware, sim_isaac, and
gazebo+moveit): each now has exactly one system declaring the joint,
where sim_gazebo and sim_isaac previously had two.

Also drops the commented-out remains of an earlier attempt at this same
guard, which sat directly above.

Co-Authored-By: Claude Opus 5 <noreply@anthropic.com>
Claude-Session: https://claude.ai/code/session_01HPYCorCh7pASi2ipJFeqJb

File: kortex_description/arms/gen3_lite/6dof/urdf/kortex.ros2_control.xacro (robot description, xacro)
@@ -150,17 +150,12 @@
         <state_interface name="effort"/>
       </joint>
-      <!--<xacro:unless value="${use_fake_hardware or sim_isaac or sim_gazebo}">-->
-        <!--<xacro:unless value="${moveit_active}">-->
-        <!--
-          <joint name="${prefix}right_finger_bottom_joint">
-            <command_interface name="position"/>
-            <state_interface name="position"/>
-            <state_interface name="velocity"/>
-          </joint>
-        -->
-       <!-- </xacro:unless> -->
-      <!-- </xacro:unless> -->
-      <!--<xacro:if value="${moveit_active}">-->
-      <xacro:unless value="${use_fake_hardware}">
+      <!-- The gripper joint has exactly one owner. The gripper's own
+           ros2_control system (see gen3_lite_2f.ros2_control.xacro) claims it
+           whenever the gripper is simulated and not driven through MoveIt;
+           this condition is the complement, so the two never both declare it.
+           Declaring it twice makes the resource manager reject the whole
+           gripper system with "Tried to insert CommandInterface with already
+           existing key". -->
+      <xacro:unless value="${(use_fake_hardware or sim_gazebo or sim_isaac) and not moveit_active}">
         <joint name="${prefix}right_finger_bottom_joint">
           <command_interface name="position"/>
@@ -169,5 +164,4 @@
         </joint>
       </xacro:unless>
-      <!--</xacro:if>-->
     </ros2_control>
   </xacro:macro>
